File: pcb/pskeeb.kicad_sch (KiCad schematic)
At the start: 29 parts, among them K11 KEYSW, K12 KEYSW, K13 KEYSW, K14 KEYSW, K15 KEYSW, K21 KEYSW, K22 KEYSW, K23 KEYSW, K24 KEYSW, K25 KEYSW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

Commit message: feat: first production
Connections:
- net joystick_btn: now also U1.17 (PB9)
- net joystick_x: now also R1.2, U2.4 (CLK)
- net joystick_y: now also R2.2, U2.5 (DAT)
- net k25: now also U1.16 (PB8); no longer U1.25 (RES)
- removed net ps/2_clk: R1.2, U1.17 (PB9), U2.4 (CLK)
- removed net ps/2_dat: R2.2, U1.16 (PB8), U2.5 (DAT)
- no-connect marks 10 -> 11
Changed lines of the file:
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@@
 (kicad_sch (version 20211123) (generator eeschema)
   (paper "A4")
+  (junction (at 96.52 107.315) (diameter 0) (color 0 0 0 0)
+  )
+  (junction (at 96.52 109.855) (diameter 0) (color 0 0 0 0)
+  )
   (junction (at 223.52 48.26) (diameter 0) (color 0 0 0 0)
   )
@@
   (junction (at 223.52 59.69) (diameter 0) (color 0 0 0 0)
   )
+  (no_connect (at 89.535 112.395))
   (no_connect (at 89.535 84.455))
   (no_connect (at 89.535 122.555))
@@
     (stroke (width 0) (type default) (color 0 0 0 0))
   )
+  (wire (pts (xy 96.52 107.315) (xy 102.235 107.315))
+    (stroke (width 0) (type default) (color 0 0 0 0))
+  )
   (wire (pts (xy 185.42 119.38) (xy 190.5 119.38))
     (stroke (width 0) (type default) (color 0 0 0 0))
   )
+  (wire (pts (xy 96.52 107.315) (xy 96.52 104.775))
+    (stroke (width 0) (type default) (color 0 0 0 0))
+  )
   (wire (pts (xy 231.14 38.1) (xy 233.68 38.1))
     (stroke (width 0) (type default) (color 0 0 0 0))
@@
     (stroke (width 0) (type default) (color 0 0 0 0))
   )
+  (wire (pts (xy 96.52 112.395) (xy 102.235 112.395))
+    (stroke (width 0) (type default) (color 0 0 0 0))
+  )
   (wire (pts (xy 250.825 61.595) (xy 250.825 63.5))
     (stroke (width 0) (type default) (color 0 0 0 0))
@@
     (stroke (width 0) (type default) (color 0 0 0 0))
   )
+  (wire (pts (xy 96.52 109.855) (xy 96.52 112.395))
+    (stroke (width 0) (type default) (color 0 0 0 0))
+  )
   (wire (pts (xy 41.275 107.315) (xy 48.895 107.315))
     (stroke (width 0) (type default) (color 0 0 0 0))
   )
+  (wire (pts (xy 102.235 109.855) (xy 96.52 109.855))
+    (stroke (width 0) (type default) (color 0 0 0 0))
+  )
   (wire (pts (xy 233.68 38.1) (xy 237.49 38.1))
     (stroke (width 0) (type default) (color 0 0 0 0))
@@
     (stroke (width 0) (type default) (color 0 0 0 0))
   )
+  (wire (pts (xy 96.52 104.775) (xy 102.235 104.775))
+    (stroke (width 0) (type default) (color 0 0 0 0))
+  )
   (wire (pts (xy 249.555 146.05) (xy 242.57 146.05))
     (stroke (width 0) (type default) (color 0 0 0 0))
@@
     (stroke (width 0) (type default) (color 0 0 0 0))
   )
+  (wire (pts (xy 96.52 107.315) (xy 89.535 107.315))
+    (stroke (width 0) (type default) (color 0 0 0 0))
+  )
   (wire (pts (xy 250.825 57.785) (xy 250.825 59.69))
     (stroke (width 0) (type default) (color 0 0 0 0))
@@
     (stroke (width 0) (type default) (color 0 0 0 0))
   )
+  (wire (pts (xy 96.52 109.855) (xy 89.535 109.855))
+    (stroke (width 0) (type default) (color 0 0 0 0))
+  )
   (wire (pts (xy 83.82 137.16) (xy 88.9 137.16))
     (stroke (width 0) (type default) (color 0 0 0 0))
@@
     (effects (font (size 1.27 1.27)) (justify left bottom))
   )
-  (label "k25" (at 89.535 112.395 0)
-    (effects (font (size 1.27 1.27)) (justify left bottom))
-  )
   (label "k31" (at 89.535 114.935 0)
     (effects (font (size 1.27 1.27)) (justify left bottom))
@@
     (effects (font (size 1.27 1.27)) (justify left bottom))
   )
+  (label "joystick_btn" (at 48.895 114.935 180)
+    (effects (font (size 1.27 1.27)) (justify right bottom))
+  )
   (label "k12" (at 89.535 86.995 0)
     (effects (font (size 1.27 1.27)) (justify left bottom))
@@
     (effects (font (size 1.27 1.27)) (justify left bottom))
   )
-  (label "joystick_x" (at 89.535 109.855 0)
+  (label "joystick_x" (at 102.235 109.855 0)
     (effects (font (size 1.27 1.27)) (justify left bottom))
   )
@@
     (effects (font (size 1.27 1.27)) (justify left bottom))
   )
-  (label "ps{slash}2_dat" (at 48.895 112.395 180)
-    (effects (font (size 1.27 1.27)) (justify right bottom))
+  (label "ps{slash}2_clk" (at 102.235 112.395 0)
+    (effects (font (size 1.27 1.27)) (justify left bottom))
   )
   (label "k15" (at 241.3 88.9 0)
     (effects (font (size 1.27 1.27)) (justify left bottom))
   )
+  (label "k25" (at 48.895 112.395 180)
+    (effects (font (size 1.27 1.27)) (justify right bottom))
+  )
   (label "k21" (at 89.535 97.155 0)
     (effects (font (size 1.27 1.27)) (justify left bottom))
@@
     (effects (font (size 1.27 1.27)) (justify right bottom))
   )
-  (label "joystick_y" (at 89.535 107.315 0)
+  (label "joystick_y" (at 102.235 107.315 0)
     (effects (font (size 1.27 1.27)) (justify left bottom))
   )
@@
     (effects (font (size 1.27 1.27)) (justify left bottom))
   )
+  (label "ps{slash}2_dat" (at 102.235 104.775 0)
+    (effects (font (size 1.27 1.27)) (justify left bottom))
+  )
   (label "k22" (at 157.48 104.14 0)
     (effects (font (size 1.27 1.27)) (justify left bottom))
@@
     (effects (font (size 1.27 1.27)) (justify left bottom))
   )
-  (label "ps{slash}2_clk" (at 48.895 114.935 180)
-    (effects (font (size 1.27 1.27)) (justify right bottom))
-  )
   (label "k42" (at 48.895 102.235 180)
