File: pcbs/pskeeb.kicad_sch (KiCad schematic)
At the start: 29 parts, among them K11 KEYSW, K12 KEYSW, K13 KEYSW, K14 KEYSW, K15 KEYSW, K21 KEYSW, K22 KEYSW, K23 KEYSW, K24 KEYSW, K25 KEYSW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

Commit message: fix: bigger resistor / ec11 share holes / usb fit
Parts:
- removed U2: PS/2_Trackpoint, Connector_PinHeader_2.54mm:PinHeader_1x05_P2.54mm_Vertical, symbol trackpoint:PS/2_Trackpoint
- removed U3: JoyStick, Connector_PinHeader_2.54mm:PinHeader_1x05_P2.54mm_Vertical, symbol joystick:JoyStick
- added K1: KEYSW, Resistor_SMD:R_0201_0603Metric_Pad0.64x0.40mm_HandSolder, symbol keyboard_parts:KEYSW
- added U2: trackpoint/joystick, Connector_JST:JST_GH_BM05B-GHS-TBT_1x05-1MP_P1.25mm_Vertical, symbol pskeeb-components:trackpoint/joystick
- R1, R2, R3: footprint Resistor_THT:R_Axial_DIN0204_L3.6mm_D1.6mm_P5.08mm_Horizontal -> Resistor_THT:R_Axial_DIN0207_L6.3mm_D2.5mm_P10.16mm_Horizontal
Connections:
- net +5V: now also U2.5 (VCC)
- net GND: now also U2.4 (GND)
- net joystick_btn: now also K1.2
- net RST/BTN: now reaches C1.2, R3.1
- net RST/BTN: now also K1.1, U2.1 (RST/BTN)
- net joystick_x renamed CLK/X
- net CLK/X: now also U2.3 (CLK/X)
- net joystick_y renamed DAT/Y
- net DAT/Y: now also U2.2 (DAT/Y)
Other:
- moved on the sheet: C1, R1, R2, R3
