File: trackball1_hugebug/pcb/trackball1_hugebug.kicad_sch (KiCad schematic)
At the start: 18 parts, among them J1 Conn_01x03, J10 Conn_01x03, J11 Conn_01x03, J2 Conn_01x03, J3 Conn_01x03, J4 Conn_01x03, J5 Conn_01x08, J6 Conn_01x02, J7 Conn_01x02, J8 Conn_01x03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

Commit message: refactor: increase footprint pads for easier soldering
Parts:
- removed J5: Conn_01x08, Connector_FFC-FPC:Hirose_FH12-8S-0.5SH_1x08-1MP_P0.50mm_Horizontal, symbol Connector_Generic:Conn_01x08
- removed SW1, SW2, SW3, SW4: SW_SPDT, kwkb-footprint:MouseSwitch, symbol Switch:SW_SPDT
- added J5: Conn_01x06, Connector_JST:JST_GH_BM06B-GHS-TBT_1x06-1MP_P1.25mm_Vertical, symbol Connector_Generic:Conn_01x06
- added SW1, SW2, SW3, SW4: SW_SPDT_312, kwkb-footprint:MouseSwitch, symbol Switch:SW_SPDT_312
Connections:
- net GND: now also J1.2 (Pin_2), J2.2 (Pin_2), J3.2 (Pin_2), J4.2 (Pin_2), J5.2 (Pin_2); no longer J1.3 (Pin_3), J10.3 (Pin_3), J11.3 (Pin_3), J2.3 (Pin_3), J3.3 (Pin_3), J4.3 (Pin_3), J8.3 (Pin_3), J9.3 (Pin_3)
- net MOTION: now also J5.6 (Pin_6)
- net SCLK: now also J5.5 (Pin_5)
- net SDIO: now also J5.4 (Pin_4)
- net VIN: now also J5.1 (Pin_1)
- net btn1: now also J1.3 (Pin_3); no longer J1.2 (Pin_2)
- net btn2: now also J2.3 (Pin_3); no longer J2.2 (Pin_2)
- net btn3: now also J3.3 (Pin_3); no longer J3.2 (Pin_2)
- net btn4: now also J4.3 (Pin_3); no longer J4.2 (Pin_2)
- net nCS: now also J5.3 (Pin_3)
- net at J9.1 (Pin_1): now also SW2.1 (B)
- net at J9.2 (Pin_2): now also SW2.2 (C)
- net at J11.1 (Pin_1): now also SW4.1 (B)
- net at J11.2 (Pin_2): now also SW4.2 (C)
- net at J8.1 (Pin_1): now also SW1.1 (B)
- net at J8.2 (Pin_2): now also SW1.2 (C)
- net at J10.1 (Pin_1): now also SW3.1 (B)
- net at J10.2 (Pin_2): now also SW3.2 (C)
- new net: J10.3 (Pin_3), SW3.3 (A)
- new net: J11.3 (Pin_3), SW4.3 (A)
- new net: J8.3 (Pin_3), SW1.3 (A)
- new net: J9.3 (Pin_3), SW2.3 (A)
- no-connect marks 7 -> 5
Other:
- moved on the sheet: J3, J4, J8
